File: Hardware/PCB/harp behavior.brd (EAGLE design)
At the start: 87 x 83.5 mm, 174 parts, among them IC1 USBLC6-2SC6, IC10 OPA365, IC12 SN74LVC1G125, IC13 M74VHC1GT50DTT1G, IC14 SN74LVC1G125, IC15 M74VHC1GT50DTT1G, IC16 SN74LVC1G125, IC17 M74VHC1GT50DTT1G, IC2 DC-DC-SIP-5, IC3 LP5907MFX-3.3, IC4 FT232RL, IC5 TPS78630DCQ, IC6 M74VHC1GT50DTT1G, IC7 XMEGA-A1TQFP, IC9 LP5907MFX-3.3, J1 22-05-7038-03, J2 Port 0, J3 Port 1, J4 Port 2, Q1 MOSFET-NCHANNELSOT323, Q10 BC817-40W, Q13 MOSFET-NCHANNELSOT323, Q14 MOSFET-NCHANNELSOT323, Q15 MOSFET-NCHANNELSOT323, Q3 MOSFET-NCHANNELSOT323, Q5 BC817-40W, Q6 BC817-40W, Q9 BC817-40W, X1 CON_3.5MM_1X2, X2 CON_3.5MM_1X2, X3 CON_3.5MM_1X4, X4 CON_3.5MM_1X3, X5 CON_3.5MM_1X3

Commit message: Organized files for PCB version 2.0.
Parts:
- removed F1: 1A FB, rcl:R0603
- added C50, C51: 15nF 5%, rcl:C0402
- added C52, C53: 100nF, rcl:C0402
- added IC18: OPA365, CNP-ics 2:SOT23-5
- added IC19: SN74LVC1G125, My_library 0v2:SOT23-5
- added R48, R49: 10k 1%, rcl:R0402
- added R50: 24k, rcl:R0402
- added R51: 15k, rcl:R0402
- added R52: 100k, rcl:R0402
- D1, D2, D3, D4: device diode:SOD323-R -> CNP-miscellaneous:SOD-323-DIODE
- IC5: value TPS78630DCQ -> TPS78601SON; device CNP:SOT223-6 -> CNP-ics 1:SON-8
- L1: device CNP-miscellaneous:IND_LPS4012 -> CNP-miscellaneous:IND_LPS4012_V2
- OSC1: value (none) -> OSCILLATOR
- R14: value 16k -> 15k
- X3: value CON_3.5MM_1X4 -> CON_3.5MM_1X3; device CNP-connectors:CON_3.5MM_1X4 -> CNP-connectors:CON_3.5MM_1X3
- X4: value CON_3.5MM_1X3 -> CON_3.5MM_1X6; device CNP-connectors:CON_3.5MM_1X3 -> CNP-connectors:CON_3.5MM_1X6
- X5: value CON_3.5MM_1X3 -> CON_3.5MM_1X4; device CNP-connectors:CON_3.5MM_1X3 -> CNP-connectors:CON_3.5MM_1X4
- moved X3 35.7 mm to (75.5, 39.5), turned to 270 degrees
- moved X4 15.2 mm to (78.0, 19.1)
- moved X5 11.4 mm to (68.5, 4.50), turned to 180 degrees
- moved U$2 11.0 mm to (73.5, 32.5)
- moved U$6 11.0 mm to (73.5, 32.5)
- moved R25 10.0 mm to (79.5, 27.5)
- moved R31 10.0 mm to (79.5, 24.0)
- moved Q5 6.50 mm to (68.8, 29.4)
- moved Q11 6.50 mm to (68.0, 24.0)
- moved Q7 6.50 mm to (68.0, 31.0)
- moved Q9 6.50 mm to (68.8, 22.1)
- moved R23 6.50 mm to (69.7, 32.4)
- moved R27 6.50 mm to (64.5, 22.7)
- moved R29 6.50 mm to (69.7, 25.3)
- moved R21 6.50 mm to (64.4, 30.0)
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Connections:
- new net ADC1: C51.2, IC7.97, R49.2
- new net ADC1_IN: R50.2, X3.P1
- new net DI3: IC19.2, R52.1, X3.P3
- new net IN03: IC19.4, IC7.55
- new net N$19: IC18.1, IC18.4, R48.1
- new net N$29: IC18.3, R50.1, R51.2
- net +12V: now also JACK.P1; no longer F1.1
- net +5V: now also IC5.P3, IC5.P4, X5.P1; no longer IC5.P$4, X3.P1
- net ADC0_IN: now also X5.P3; no longer X3.P3
- net DO0: now also X4.P5; no longer X5.P2
- net DO1: now also X4.P4; no longer X5.P1
- net GND: now also C50.1, C51.1, C52.2, C53.2, IC18.2, IC19.1, IC19.3, IC5.P6, IC5.P9, R51.1, R52.2, X4.P6, X5.P2, X5.P4; no longer IC5.P$3, IC5.P$6, X3.P4, X5.P3
- net N$18: now also C50.2, R48.2, R49.1; no longer F1.2, JACK.P1
- net N$20: now also IC5.P5; no longer IC5.P$5
- net P5.45V: now also IC5.P1, IC5.P2, IC5.P8; no longer IC5.P$1, IC5.P$2
- net VCCIO: now also C53.1, IC19.5, IC7.65
- net VDD: now also C52.1, IC18.5
Routing:
- net +5V: track 474.8 -> 438.3 mm, vias 20 -> 19
- net ADC1: track 0.00 -> 28.5 mm, vias 0 -> 2
- net DI3: track 0.00 -> 27.9 mm, vias 0 -> 1
- net VCCIO: track 294.4 -> 320.7 mm, vias 19 -> 21
- net VDD: track 101.4 -> 109.3 mm
- net P5.45V: track 27.3 -> 34.4 mm, vias 2 -> 0
- net GND: track 8.00 -> 1.50 mm, vias 166 -> 177
- net TOG_D03: track 34.7 -> 41.2 mm
- net TOG_D02: track 31.9 -> 37.6 mm
- net N$19: track 0.00 -> 5.60 mm
- net IN03: track 0.00 -> 5.25 mm
- net LED_DATA: track 76.3 -> 71.8 mm
- net ADC1_IN: track 0.00 -> 4.46 mm
- net N$20: track 7.27 -> 11.5 mm, vias 0 -> 2
- net N$29: track 0.00 -> 4.19 mm, vias 0 -> 1
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Other:
- board text added: "+"
- board text added: "."
- board text added: "5V Inputs"
- board text added: "AD0"
- board text added: "AD1"
- board text added: "DI3"
- board text added: "Licensed under the TAPR Open Hardware License (www.tapr.org/OHL) Copyright 2021 Artur Silva and Filipe Carvalho"
- board text added: "harp behavior v2.0"
- board text removed: "ADC"
- board text removed: "Licensed under the TAPR Open Hardware License (www.tapr.org/OHL) Copyright 2017 Artur Silva and Filipe Carvalho"
- board text removed: "harp behavior v1.2"
