File: Hardware/PCB/harp behavior.sch (EAGLE design)
At the start: 166 parts, among them IC1 USBLC6-2SC6, IC10 OPA365, IC11 AD8041R, IC12 SN74LVC1G125, IC13 M74VHC1GT50DTT1G, IC14 SN74LVC1G125, IC15 M74VHC1GT50DTT1G, IC16 SN74LVC1G125, IC17 M74VHC1GT50DTT1G, IC2 DC-DC-SIP-5, IC3 LP5907MFX-3.3, IC4 FT232RL, IC5 TPS78630DCQ, IC6 M74VHC1GT50DTT1G, IC7 XMEGA-A1TQFP, IC8 AD8041R, IC9 LP5907MFX-3.3, J1 22-05-7038-03, J2 Port 0, J3 Port 1, J4 Port 2, Q1 MOSFET-NCHANNELSOT323, Q10 BC817-40W, Q13 MOSFET-NCHANNELSOT323, Q14 MOSFET-NCHANNELSOT323, Q15 MOSFET-NCHANNELSOT323, Q3 MOSFET-NCHANNELSOT323, Q5 BC817-40W, Q6 BC817-40W, Q9 BC817-40W, X1 CON_3.5MM_1X2, X2 CON_3.5MM_1X2, X3 CON_3.5MM_1X4, X4 CON_3.5MM_1X3, X5 CON_3.5MM_1X3

Commit message: Organized files for PCB version 2.0.
Parts:
- removed F1: 1A FB, rcl:R-EU_R0603
- added C50, C51: 15nF 5%, rcl:C-EUC0402
- added C52, C53: 100nF, rcl:C-EUC0402
- added IC18: OPA365, CNP-ics 2:OPA365
- added IC19: SN74LVC1G125, My_library 0v2:SN74LVC1G125
- added R48, R49: 10k 1%, rcl:R-EU_R0402
- added R50: 24k, rcl:R-EU_R0402
- added R51: 15k, rcl:R-EU_R0402
- added R52: 100k, rcl:R-EU_R0402
- D1, D2, D3, D4: device diode:DIODE-SOD323-R -> CNP-miscellaneous:DIODE
- IC5: value TPS78630DCQ -> TPS78601SON; device CNP:TPS795XX -> CNP-ics 1:TPS78601SON
- L1: device CNP-miscellaneous:INDLPS4012 -> CNP-miscellaneous:INDLPS4012_L
- R14: value 16k -> 15k
- X3: value CON_3.5MM_1X4 -> CON_3.5MM_1X3; device CNP-connectors:CON_3.5MM_1X4 -> CNP-connectors:CON_3.5MM_1X3
- X4: value CON_3.5MM_1X3 -> CON_3.5MM_1X6; device CNP-connectors:CON_3.5MM_1X3 -> CNP-connectors:CON_3.5MM_1X6
- X5: value CON_3.5MM_1X3 -> CON_3.5MM_1X4; device CNP-connectors:CON_3.5MM_1X3 -> CNP-connectors:CON_3.5MM_1X4
Connections:
- new net ADC1: C51.2, IC7.PA2(ADCA2), R49.2
- new net ADC1_IN: R50.2, X3.1
- new net DI3: IC19.P$2, R52.1, X3.3
- new net IN03: IC19.P$4, IC7.PH0(!WE!)
- new net N$19: IC18.-IN, IC18.OUT, R48.1
- new net N$29: IC18.+IN, R50.1, R51.2
- net +12V: now also JACK.1; no longer F1.1
- net +5V: now also X5.1; no longer X3.1
- net ADC0_IN: now also X5.3; no longer X3.3
- net DO0: now also X4.5; no longer X5.2
- net DO1: now also X4.4; no longer X5.1
- net GND: now also C50.1, C51.1, C52.2, C53.2, IC18.V-, IC19.P$1, IC19.P$3, R51.1, R52.2, X4.6, X5.2, X5.4; no longer X3.4, X5.3
- net N$18: now also C50.2, R48.2, R49.1; no longer F1.2, JACK.1
- net VCCIO: now also C53.1, IC19.P$5, IC7.PJ0(D0/A0/A8)
- net VDD: now also C52.1, IC18.V+
Other:
- note added: "Licensed under the TAPR Open Hardware License (www.tapr.org/OHL) Copyright 2021 Artur Silva and Filipe Carvalho"
- note removed: "Licensed under the TAPR Open Hardware License (www.tapr.org/OHL) Copyright 2017 Artur Silva and Filipe Carvalho"
- note removed: "TPS78601DCQ"
- moved on the sheet: C33, C34, C35, C36, C37, C38, C39, C40, C41, C42, C43, IC10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
